Commit message: Fix mesh file paths

File: iit-cogimon/model.urdf (robot description, URDF)
Before this commit: robot cogimon, 36 links, 35 joints
Links:
- link DWL: geometry collision mesh filename=model://iit-cogimon/meshes/simple/TorsoRoll.stl scale=0.001 0.001 0.001; visual mesh filename=model://iit-cogimon/meshes/TorsoRoll.stl scale=0.001 0.001 0.001
- link LFoot: geometry collision box size=0.21 0.11 0.015; visual mesh filename=model://iit-cogimon/meshes/Foot.stl scale=0.001 0.001 0.001
- link LFootmot: geometry collision mesh filename=model://iit-cogimon/meshes/simple/AnklePitch.stl scale=0.001 0.001 0.001; visual mesh filename=model://iit-cogimon/meshes/AnklePitch.stl scale=0.001 0.001 0.001
- link LHipMot: geometry collision mesh filename=model://iit-cogimon/meshes/simple/HipRoll.stl scale=0.001 0.001 0.001; visual mesh filename=model://iit-cogimon/meshes/HipRoll.stl scale=0.001 0.001 0.001
- link LLowLeg: geometry collision mesh filename=model://iit-cogimon/meshes/simple/KneePitch.stl scale=0.001 0.001 0.001; visual mesh filename=model://iit-cogimon/meshes/KneePitch.stl scale=0.001 0.001 0.001
- link LThighLowLeg: geometry collision mesh filename=model://iit-cogimon/meshes/simple/HipYaw.stl scale=0.001 0.001 0.001; visual mesh filename=model://iit-cogimon/meshes/HipYaw.stl scale=0.001 0.001 0.001
- link LThighUpLeg: geometry collision mesh filename=model://iit-cogimon/meshes/simple/HipPitch.stl scale=0.001 0.001 0.001; visual mesh filename=model://iit-cogimon/meshes/HipPitch.stl scale=0.001 0.001 0.001
- link RFoot: geometry collision box size=0.21 0.11 0.015; visual mesh filename=model://iit-cogimon/meshes/Foot.stl scale=0.001 0.001 0.001
- link RFootmot: geometry collision mesh filename=model://iit-cogimon/meshes/simple/AnklePitch.stl scale=0.001 0.001 0.001; visual mesh filename=model://iit-cogimon/meshes/AnklePitch.stl scale=0.001 0.001 0.001
- link RHipMot: geometry collision mesh filename=model://iit-cogimon/meshes/simple/HipRoll.stl scale=0.001 -0.001 0.001; visual mesh filename=model://iit-cogimon/meshes/HipRoll.stl scale=0.001 -0.001 0.001
- link RLowLeg: geometry collision mesh filename=model://iit-cogimon/meshes/simple/KneePitch.stl scale=0.001 -0.001 0.001; visual mesh filename=model://iit-cogimon/meshes/KneePitch.stl scale=0.001 -0.001 0.001
- link RThighLowLeg: geometry collision mesh filename=model://iit-cogimon/meshes/simple/HipYaw.stl scale=0.001 -0.001 0.001; visual mesh filename=model://iit-cogimon/meshes/HipYaw.stl scale=0.001 -0.001 0.001
- link RThighUpLeg: geometry collision mesh filename=model://iit-cogimon/meshes/simple/HipPitch.stl scale=0.001 -0.001 0.001; visual mesh filename=model://iit-cogimon/meshes/HipPitch.stl scale=0.001 -0.001 0.001
- link Waist: geometry collision mesh filename=model://iit-cogimon/meshes/simple/Waist.stl scale=0.001 0.001 0.001; visual mesh filename=model://iit-cogimon/meshes/Waist.stl scale=0.001 0.001 0.001
- link pennacchio: geometry collision mesh filename=model://iit-cogimon/meshes/simple/Pennacchio.stl scale=0.001 0.001 0.001; visual mesh filename=model://iit-cogimon/meshes/Pennacchio.stl scale=0.001 0.001 0.001
