Commit message: Adjust mesh file paths

File: franka/model.urdf (robot description, URDF)
Before this commit: robot panda, 10 links, 9 joints
Links:
- link panda_link0: geometry collision mesh filename=model://franka/meshes/link0_collision.STL; visual mesh filename=model://franka/meshes/link0.dae
- link panda_link1: geometry collision mesh filename=model://franka/meshes/link1_collision.STL; visual mesh filename=model://franka/meshes/link1.dae
- link panda_link2: geometry collision mesh filename=model://franka/meshes/link2_collision.STL; visual mesh filename=model://franka/meshes/link2.dae
- link panda_link3: geometry collision mesh filename=model://franka/meshes/link3_collision.STL; visual mesh filename=model://franka/meshes/link3.dae
- link panda_link4: geometry collision mesh filename=model://franka/meshes/link4_collision.STL; visual mesh filename=model://franka/meshes/link4.dae
- link panda_link5: geometry collision mesh filename=model://franka/meshes/link5_collision.STL; visual mesh filename=model://franka/meshes/link5.dae
- link panda_link6: geometry collision mesh filename=model://franka/meshes/link6_collision.STL; visual mesh filename=model://franka/meshes/link6.dae
- link panda_link7: geometry collision mesh filename=model://franka/meshes/link7_collision.STL; visual mesh filename=model://franka/meshes/link7.dae
